File: PROTORS_STM32F1/PROTORS_STM32F1.sch (KiCad schematic (older format))
At the start: 33 parts, among them J1 USB_B_Mini, J2 ST-LINK, J3 PINS_1, J4 PINS_2, U1 STM32F103C8Tx, U2 AMS1117-3.3, Y1 8MHz, Y2 32.768kHz

Commit message: Update board
Parts:
- C13, C14: footprint (none) -> Capacitor_SMD:C_1206_3216Metric
- D1: footprint (none) -> Diode_SMD:D_SMA
- J2: footprint Connector_JST:JST_SH_SM04B-SRSS-TB_1x04-1MP_P1.00mm_Horizontal -> Connector_PinHeader_2.54mm:PinHeader_1x04_P2.54mm_Vertical
- J3, J4: footprint (none) -> Connector_PinHeader_2.54mm:PinHeader_2x10_P2.54mm_Vertical
- JP1, JP2, JP3: footprint (none) -> Jumper:SolderJumper-2_P1.3mm_Open_Pad1.0x1.5mm
Connections:
- net +3V3: now also J4.1 (Pin_1); no longer J4.2 (Pin_2)
- net +5V: now also J3.2 (Pin_2); no longer J3.1 (Pin_1)
- net GND: now also J3.1 (Pin_1), J3.19 (Pin_19), J4.18 (Pin_18), J4.2 (Pin_2); no longer J3.2 (Pin_2), J3.20 (Pin_20), J4.1 (Pin_1), J4.17 (Pin_17)
- net PA_0: now also J3.20 (Pin_20); no longer J3.19 (Pin_19)
- net PA_1: now also J3.18 (Pin_18); no longer J3.17 (Pin_17)
- net PA_10: now also J4.3 (Pin_3); no longer J4.4 (Pin_4)
- net PA_11: now also J4.6 (Pin_6); no longer J4.5 (Pin_5)
- net PA_12: now also J4.5 (Pin_5); no longer J4.6 (Pin_6)
- net PA_13: now also J4.8 (Pin_8); no longer J4.7 (Pin_7)
- net PA_14: now also J4.7 (Pin_7); no longer J4.8 (Pin_8)
- net PA_15: now also J4.10 (Pin_10); no longer J4.9 (Pin_9)
- net PA_2: now also J3.17 (Pin_17); no longer J3.18 (Pin_18)
- net PA_3: now also J3.16 (Pin_16); no longer J3.15 (Pin_15)
- net PA_4: now also J3.15 (Pin_15); no longer J3.16 (Pin_16)
- net PA_5: now also J3.14 (Pin_14); no longer J3.13 (Pin_13)
- net PA_6: now also J3.13 (Pin_13); no longer J3.14 (Pin_14)
- net PA_7: now also J3.12 (Pin_12); no longer J3.11 (Pin_11)
- net PA_8: now also J3.3 (Pin_3); no longer J3.4 (Pin_4)
- net PA_9: now also J4.4 (Pin_4); no longer J4.3 (Pin_3)
- net PB_0: now also J3.11 (Pin_11); no longer J3.12 (Pin_12)
- net PB_1: now also J3.10 (Pin_10); no longer J3.9 (Pin_9)
- net PB_10: now also J3.9 (Pin_9); no longer J3.10 (Pin_10)
- net PB_11: now also J3.8 (Pin_8); no longer J3.7 (Pin_7)
- net PB_12: now also J3.7 (Pin_7); no longer J3.8 (Pin_8)
- net PB_13: now also J3.6 (Pin_6); no longer J3.5 (Pin_5)
- net PB_14: now also J3.5 (Pin_5); no longer J3.6 (Pin_6)
- net PB_15: now also J3.4 (Pin_4); no longer J3.3 (Pin_3)
- net PB_3: now also J4.9 (Pin_9); no longer J4.10 (Pin_10)
- net PB_4: now also J4.12 (Pin_12); no longer J4.11 (Pin_11)
- net PB_5: now also J4.11 (Pin_11); no longer J4.12 (Pin_12)
- net PB_6: now also J4.14 (Pin_14); no longer J4.13 (Pin_13)
- net PB_7: now also J4.13 (Pin_13); no longer J4.14 (Pin_14)
- net PB_8: now also J4.16 (Pin_16); no longer J4.15 (Pin_15)
- net PB_9: now also J4.15 (Pin_15); no longer J4.16 (Pin_16)
- net PC_13: now also J4.17 (Pin_17); no longer J4.18 (Pin_18)
Changed lines of the file:
@@
 encoding utf-8
 Sheet 1 1
-Title "PROTORS_STM32F1_001"
+Title "PROTORS_STM32F1"
 Date "2020-04-27"
 Rev "2"
-Comp "PROTORS"
-Comment1 "PROTORS_STM32F1"
+Comp "Protors"
+Comment1 "PROTORS_STM32"
 Comment2 "Veljko Petrović"
 Comment3 "Veljko Petrović"
@@
 F 0 "J2" H 1930 4592 50  0000 L CNN
 F 1 "ST-LINK" H 1930 4501 50  0000 L CNN
-F 2 "Connector_JST:JST_SH_SM04B-SRSS-TB_1x04-1MP_P1.00mm_Horizontal" H 1850 4600 50  0001 C CNN
+F 2 "Connector_PinHeader_2.54mm:PinHeader_1x04_P2.54mm_Vertical" H 1850 4600 50  0001 C CNN
 F 3 "~" H 1850 4600 50  0001 C CNN
 	1    1850 4600
@@
 L power:GND #PWR04
 U 1 1 5E8AE6F9
-P 1600 5000
-F 0 "#PWR04" H 1600 4750 50  0001 C CNN
-F 1 "GND" H 1605 4827 50  0000 C CNN
-F 2 "" H 1600 5000 50  0001 C CNN
-F 3 "" H 1600 5000 50  0001 C CNN
-	1    1600 5000
+P 1550 5000
+F 0 "#PWR04" H 1550 4750 50  0001 C CNN
+F 1 "GND" H 1555 4827 50  0000 C CNN
+F 2 "" H 1550 5000 50  0001 C CNN
+F 3 "" H 1550 5000 50  0001 C CNN
+	1    1550 5000
 	1    0    0    -1
 $EndComp
@@
 L power:+3V3 #PWR02
 U 1 1 5E8AE6FF
-P 1400 5000
-F 0 "#PWR02" H 1400 4850 50  0001 C CNN
-F 1 "+3V3" H 1415 5173 50  0000 C CNN
-F 2 "" H 1400 5000 50  0001 C CNN
-F 3 "" H 1400 5000 50  0001 C CNN
-	1    1400 5000
+P 1350 5000
+F 0 "#PWR02" H 1350 4850 50  0001 C CNN
+F 1 "+3V3" H 1365 5173 50  0000 C CNN
+F 2 "" H 1350 5000 50  0001 C CNN
+F 3 "" H 1350 5000 50  0001 C CNN
+	1    1350 5000
 	-1   0    0    1
 $EndComp
 Wire Wire Line
-	1400 5000 1400 4500
-Wire Wire Line
-	1400 4500 1650 4500
+	1350 5000 1350 4500
+Wire Wire Line
+	1350 4500 1650 4500
 Text GLabel 2900 1400 0    50   UnSpc ~ 0
 HSE_1
@@
 Wire Wire Line
 	2900 3000 3050 3000
-Wire Wire Line
-	1650 4600 1250 4600
 Text GLabel 2900 2100 0    50   BiDi ~ 0
 PB_0
@@
 F 0 "D1" H 1950 6134 50  0000 C CNN
 F 1 "SS14" H 1950 6225 50  0000 C CNN
-F 2 "" H 1950 6350 50  0001 C CNN
+F 2 "Diode_SMD:D_SMA" H 1950 6350 50  0001 C CNN
 F 3 "~" H 1950 6350 50  0001 C CNN
 	1    1950 6350
@@
 Text GLabel 1850 6650 2    50   BiDi ~ 0
 PA_11
-Wire Wire Line
-	1600 5000 1600 4800
-Wire Wire Line
-	1600 4800 1650 4800
 Text GLabel 1250 4600 0    50   BiDi ~ 0
 PA_13
 Text GLabel 1250 4700 0    50   BiDi ~ 0
 PA_14
-Wire Wire Line
-	1250 4700 1650 4700
 Text GLabel 2900 1200 0    50   Input ~ 0
 BOOT_0
@@
 F 0 "JP2" H 6750 4355 50  0000 C CNN
 F 1 "BOOT0" H 6750 4264 50  0000 C CNN
-F 2 "" H 6750 4150 50  0001 C CNN
+F 2 "Jumper:SolderJumper-2_P1.3mm_Open_Pad1.0x1.5mm" H 6750 4150 50  0001 C CNN
 F 3 "~" H 6750 4150 50  0001 C CNN
 	1    6750 4150
@@
 F 0 "JP3" H 6750 5105 50  0000 C CNN
 F 1 "BOOT1" H 6750 5014 50  0000 C CNN
-F 2 "" H 6750 4900 50  0001 C CNN
+F 2 "Jumper:SolderJumper-2_P1.3mm_Open_Pad1.0x1.5mm" H 6750 4900 50  0001 C CNN
 F 3 "~" H 6750 4900 50  0001 C CNN
 	1    6750 4900
@@
 F 0 "C13" H 8968 3396 50  0000 L CNN
 F 1 "10uF" H 8968 3305 50  0000 L CNN
-F 2 "" H 8888 3200 50  0001 C CNN
+F 2 "Capacitor_SMD:C_1206_3216Metric" H 8888 3200 50  0001 C CNN
 F 3 "~" H 8850 3350 50  0001 C CNN
 	1    8850 3350
@@
 F 0 "C14" H 9968 3396 50  0000 L CNN
 F 1 "10uF" H 9968 3305 50  0000 L CNN
-F 2 "" H 9888 3200 50  0001 C CNN
+F 2 "Capacitor_SMD:C_1206_3216Metric" H 9888 3200 50  0001 C CNN
 F 3 "~" H 9850 3350 50  0001 C CNN
 	1    9850 3350
@@
 F 0 "JP1" H 6750 3555 50  0000 C CNN
 F 1 "RESET" H 6750 3464 50  0000 C CNN
-F 2 "" H 6750 3350 50  0001 C CNN
+F 2 "Jumper:SolderJumper-2_P1.3mm_Open_Pad1.0x1.5mm" H 6750 3350 50  0001 C CNN
 F 3 "~" H 6750 3350 50  0001 C CNN
 	1    6750 3350
@@
 L Connector_Generic:Conn_02x10_Odd_Even J3
 U 1 1 5F068377
-P 6950 1550
-F 0 "J3" H 7000 2167 50  0000 C CNN
-F 1 "PINS_1" H 7000 2076 50  0000 C CNN
-F 2 "" H 6950 1550 50  0001 C CNN
-F 3 "~" H 6950 1550 50  0001 C CNN
-	1    6950 1550
-	1    0    0    -1
+P 7050 1550
+F 0 "J3" H 7100 2167 50  0000 C CNN
+F 1 "PINS_1" H 7100 2076 50  0000 C CNN
+F 2 "Connector_PinHeader_2.54mm:PinHeader_2x10_P2.54mm_Vertical" H 7050 1550 50  0001 C CNN
+F 3 "~" H 7050 1550 50  0001 C CNN
+	1    7050 1550
+	-1   0    0    -1
 $EndComp
 $Comp
 L Connector_Generic:Conn_02x10_Odd_Even J4
 U 1 1 5F06964C
-P 9050 1550
-F 0 "J4" H 9100 2167 50  0000 C CNN
-F 1 "PINS_2" H 9100 2076 50  0000 C CNN
-F 2 "" H 9050 1550 50  0001 C CNN
-F 3 "~" H 9050 1550 50  0001 C CNN
-	1    9050 1550
-	1    0    0    -1
+P 9150 1550
+F 0 "J4" H 9200 2167 50  0000 C CNN
+F 1 "PINS_2" H 9200 2076 50  0000 C CNN
+F 2 "Connector_PinHeader_2.54mm:PinHeader_2x10_P2.54mm_Vertical" H 9150 1550 50  0001 C CNN
+F 3 "~" H 9150 1550 50  0001 C CNN
+	1    9150 1550
+	-1   0    0    -1
 $EndComp
 $Comp
@@
 Wire Wire Line
 	9350 2050 9450 2050
+Wire Wire Line
+	1650 4800 1550 4800
+Wire Wire Line
+	1250 4700 1650 4700
+Wire Wire Line
+	1550 4800 1550 5000
+Wire Wire Line
+	1250 4600 1650 4600
 $EndSCHEMATC
